File: PCB/Eagel/MotorSliderNoPower.brd (EAGLE design)
At the start: 147.1 x 17.8 mm, 31 parts, among them IC1 ATTINY804-SSNR, IC2 AT42QT1010, IC3 L293DD, IC4 SN74LVC1G14DBVR, X1 22-23-2021

Commit message: Update
Parts:
- moved R3 0.52 mm to (90.6, 10.0)
Routing:
- net GND: vias 29 -> 30
Changed lines of the file:
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@@
 <wire x1="91.44" y1="1.651" x2="93.726" y2="1.651" width="0.1524" layer="21"/>
 <wire x1="93.726" y1="1.651" x2="93.726" y2="5.969" width="0.1524" layer="21"/>
-<wire x1="92.202" y1="11.303" x2="92.202" y2="9.017" width="0.1524" layer="21"/>
-<wire x1="92.202" y1="9.017" x2="87.884" y2="9.017" width="0.1524" layer="21"/>
-<wire x1="87.884" y1="9.017" x2="87.884" y2="11.303" width="0.1524" layer="21"/>
-<wire x1="87.884" y1="11.303" x2="92.202" y2="11.303" width="0.1524" layer="21"/>
+<wire x1="92.71" y1="11.176" x2="92.71" y2="8.89" width="0.1524" layer="21"/>
+<wire x1="92.71" y1="8.89" x2="88.392" y2="8.89" width="0.1524" layer="21"/>
+<wire x1="88.392" y1="8.89" x2="88.392" y2="11.176" width="0.1524" layer="21"/>
+<wire x1="88.392" y1="11.176" x2="92.71" y2="11.176" width="0.1524" layer="21"/>
 <wire x1="127.127" y1="7.239" x2="129.667" y2="7.239" width="0.1524" layer="21"/>
 <wire x1="129.667" y1="7.239" x2="129.667" y2="2.667" width="0.1524" layer="21"/>
@@
 <attribute name="SPICEPREFIX" value="R" x="129.032" y="-20.955" size="1.778" layer="27" display="off"/>
 </element>
-<element name="R3" library="rcl" library_urn="urn:adsk.eagle:library:334" package="R0805" package3d_urn="urn:adsk.eagle:package:23553/2" value="100K" x="90.043" y="10.16" smashed="yes" rot="R180">
-<attribute name="NAME" x="91.059" y="12.954" size="1.27" layer="25" rot="R180"/>
-<attribute name="POPULARITY" value="86" x="29.083" y="45.72" size="1.778" layer="27" rot="R180" display="off"/>
-<attribute name="SPICEPREFIX" value="R" x="29.083" y="45.72" size="1.778" layer="27" rot="R180" display="off"/>
+<element name="R3" library="rcl" library_urn="urn:adsk.eagle:library:334" package="R0805" package3d_urn="urn:adsk.eagle:package:23553/2" value="100K" x="90.551" y="10.033" smashed="yes" rot="R180">
+<attribute name="NAME" x="91.567" y="12.827" size="1.27" layer="25" rot="R180"/>
+<attribute name="POPULARITY" value="86" x="29.591" y="45.593" size="1.778" layer="27" rot="R180" display="off"/>
+<attribute name="SPICEPREFIX" value="R" x="29.591" y="45.593" size="1.778" layer="27" rot="R180" display="off"/>
 </element>
 <element name="R4" library="rcl" library_urn="urn:adsk.eagle:library:334" package="R0805" package3d_urn="urn:adsk.eagle:package:23553/2" value="10K" x="24.13" y="13.97" smashed="yes" rot="R180">
@@
 <wire x1="40.132" y1="12.319" x2="40.132" y2="11.43" width="0.3048" layer="1"/>
 <wire x1="40.833" y1="13.02" x2="40.132" y2="12.319" width="0.3048" layer="1"/>
+<via x="83.82" y="10.922" extent="1-16" drill="0.35"/>
 </signal>
 <signal name="+5V">
@@
 <wire x1="77.47" y1="13.97" x2="77.47" y2="15.3416" width="0.3048" layer="1"/>
 <wire x1="77.47" y1="15.3416" x2="78.74" y2="16.6116" width="0.3048" layer="1"/>
-<wire x1="90.297" y1="14.351" x2="90.297" y2="11.938" width="0.3048" layer="1"/>
-<wire x1="90.297" y1="11.938" x2="90.932" y2="11.303" width="0.3048" layer="1"/>
-<wire x1="90.932" y1="11.303" x2="90.932" y2="10.221" width="0.3048" layer="1"/>
-<wire x1="90.993" y1="10.16" x2="90.932" y2="10.221" width="0.3048" layer="1"/>
+<wire x1="90.297" y1="14.351" x2="90.297" y2="12.319" width="0.3048" layer="1"/>
+<wire x1="90.297" y1="12.319" x2="90.932" y2="11.684" width="0.3048" layer="1"/>
+<wire x1="90.932" y1="11.684" x2="90.932" y2="10.602" width="0.3048" layer="1"/>
+<wire x1="91.501" y1="10.033" x2="90.932" y2="10.602" width="0.3048" layer="1"/>
 <wire x1="78.74" y1="16.6116" x2="88.0364" y2="16.6116" width="0.3048" layer="1"/>
 <wire x1="88.0364" y1="16.6116" x2="90.297" y2="14.351" width="0.3048" layer="1"/>
@@
 <wire x1="86.741" y1="10.16" x2="87.63" y2="11.049" width="0.4064" layer="1"/>
 <wire x1="87.63" y1="13.97" x2="88.646" y2="13.97" width="0.3048" layer="1"/>
-<wire x1="89.093" y1="13.523" x2="89.093" y2="10.16" width="0.3048" layer="1"/>
-<wire x1="88.646" y1="13.97" x2="89.093" y2="13.523" width="0.3048" layer="1"/>
+<wire x1="89.601" y1="13.015" x2="89.601" y2="10.033" width="0.3048" layer="1"/>
+<wire x1="88.646" y1="13.97" x2="89.601" y2="13.015" width="0.3048" layer="1"/>
 <wire x1="87.63" y1="13.97" x2="87.63" y2="3.81" width="0.8128" layer="16"/>
 </signal>
