File: PCB/Eagel/MotorFaderTB6612.V.1.0.brd (EAGLE design)
At the start: 147.1 x 17.8 mm, 31 parts, among them IC1 ATTINY804-SSNR, IC2 AT42QT1010, IC3 L293DD, IC4 SN74LVC1G14DBVR, X1 22-23-2021

Commit message: Update PCB auf 1.0
Parts:
- removed +5V, +9V: 150080RS75000, SamacSys_Parts:LEDC2012X80N
- removed IC3: L293DD, SamacSys_Parts:SOIC127P1032X265-20N
- removed LB-LED: 150080GS75000, SamacSys_Parts:LEDM2012X80N
- removed R7: 1K, rcl:R0805
- removed R9: 470R, rcl:R0805
- removed TOUCH: 150080YS75000, SamacSys_Parts:LEDC2012X80N
- removed U$2: DK8DESS, LOGOS:DK8DE_KLEIN
- removed UPDI: 0, con-lstb:MA03-1
- removed X1: 22-23-2021, con-molex:22-23-2021
- added C9: 100nF, SamacSys_Parts:C0805
- added IC5: TB6612FNG,C,8,EL, SamacSys_Parts:SOP65P760X160-24N
- added LED1, LED2: 150080GS75000, SamacSys_Parts:LEDM2012X80N
- added LED3: 150080YS75000, SamacSys_Parts:LEDC2012X80N
- added LOGO: DK8DESS, LOGOS:DK8DE_KLEIN
- added SV4: 0, con-lstb:MA03-1
- added SV5: 22-23-2021, con-molex:22-23-2021
- C5, C6: value 100nF -> 10uF; device SamacSys_Parts:C0805 -> SamacSys_Parts:T491A
- C7: device SamacSys_Parts:EEE1AA220WR -> SamacSys_Parts:T491A
- C8: value 10uF -> 100nF; device SamacSys_Parts:EEE1AA220WR -> SamacSys_Parts:C0805
- R3: value 100K -> 470R
- moved C8 74.3 mm to (117.3, 2.54)
- moved C5 66.4 mm to (44.7, 3.94), turned to 270 degrees
- moved R3 29.6 mm to (61.6, 3.68), turned to 90 degrees
- moved C7 17.3 mm to (113.2, 15.1)
- moved C6 5.97 mm to (122.9, 2.54), turned to 0 degrees
- moved R5 3.27 mm to (26.0, 4.57), turned to 180 degrees
- moved IC4 3.05 mm to (46.2, 14.1)
- moved C3 2.54 mm to (26.2, 8.64)
- moved C4 2.54 mm to (31.2, 12.4)
- moved IC2 2.54 mm to (31.2, 8.64)
- moved R4 2.54 mm to (26.2, 12.4)
- moved R1 0.81 mm to (57.3, 15.1)
- renumbered IO1 to SV1, IO2 to SV2, NEO to SV3, U$1 to FADER
Connections:
- removed net ENABLE: IC1.6, IC3.1, IC3.11
- removed net LB-LED: IC1.11, LB-LED.1
- removed net MOT-A: IC1.3, IC3.19, IC3.2
- removed net MOT-B: IC1.4, IC3.12, IC3.9
- removed net N$5: LB-LED.2, R7.1
- new net AIN1: IC1.3, IC5.21
- new net AIN2: IC1.4, IC5.22
- new net PWM: IC1.6, IC5.23
- new net STBY: IC1.11, IC5.19
- net +5V: now also C5.1, C6.1, IC5.20, SV4.2, SV5.1; no longer C6.2, IC3.20, R3.1, R7.2, UPDI.2, X1.1
- net 9V-DRIVE: now also C9.1, IC5.13, IC5.14, IC5.24, SV1.6, SV2.6; no longer C5.2, IC3.10, SV1.1, SV2.1
- net D-OUT: now also R3.1; no longer R9.1
- net GND: now also C5.2, C6.2, C9.2, IC5.10, IC5.18, IC5.3, IC5.4, IC5.9, LED1.1, LED2.1, LED3.1, SV4.3; no longer +5V.1, +9V.1, C5.1, C6.1, IC3.14, IC3.15, IC3.16, IC3.17, IC3.4, IC3.5, IC3.6, IC3.7, TOUCH.1, UPDI.3
- net INR: now also SV1.1, SV2.1; no longer R3.2, SV1.6, SV2.6
- net MOT+: now also IC5.1, IC5.2; no longer IC3.18, IC3.3
- net MOT-: now also IC5.5, IC5.6; no longer IC3.13, IC3.8
- net N$2: now also LED1.2; no longer +5V.2
- net N$3: now also LED2.2; no longer +9V.2
- net N$6: now also R3.2; no longer R9.2
- net N$9: now also LED3.2; no longer TOUCH.2
- net OPTIO: now also SV5.2; no longer X1.2
- net UPDI: now also SV4.1; no longer UPDI.1
Routing:
- net MOT-A: track 82.3 -> 0.00 mm, vias 2 -> 0
- net ENABLE: track 78.7 -> 0.00 mm, vias 2 -> 0
- net MOT-B: track 74.8 -> 0.00 mm, vias 4 -> 0
- net STBY: track 0.00 -> 68.3 mm, vias 0 -> 2
- net AIN1: track 0.00 -> 67.3 mm
- net AIN2: track 0.00 -> 65.5 mm
- net +5V: track 307.4 -> 242.1 mm, vias 0 -> 2
- net PWM: track 0.00 -> 61.9 mm
- net N$6: track 54.0 -> 4.15 mm, vias 4 -> 0
- net D-OUT: track 25.0 -> 67.3 mm, vias 0 -> 2
- net INR: track 55.1 -> 33.7 mm, vias 0 -> 1
- net 9V-DRIVE: track 82.0 -> 71.9 mm, vias 1 -> 0
- net MOT+: track 32.8 -> 40.7 mm, vias 2 -> 0
- net LB-LED: track 3.81 -> 0.00 mm
- net N$4: track 10.8 -> 7.73 mm
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Other:
- board text added: "I2C Servo Faders V1.0"
- board text added: "NEO-PIXEL-LED"
- board text added: "TOUCH"
- board text removed: "For Behringer X-Touch Fader MF100T Or Soundwell SM10001NKA0X-HA1"
