File: PCB/Eagel/MotorFaderTB6612.V.1.0.sch (EAGLE design)
At the start: 31 parts, among them IC1 ATTINY804-SSNR, IC2 AT42QT1010, IC3 L293DD, IC4 SN74LVC1G14DBVR, X1 22-23-2021

Commit message: Update PCB auf 1.0
Parts:
- removed +5V, +9V: 150080RS75000, SamacSys_Parts:150080RS75000
- removed IC3: L293DD, SamacSys_Parts:L293DD
- removed LB-LED: 150080GS75000, SamacSys_Parts:150080GS75000
- removed R7: 1K, rcl:R-EU_R0805
- removed R9: 470R, rcl:R-EU_R0805
- removed U$1: MF100T, Slider:SM10001NKA0X-HA1
- added C9: 100nF, SamacSys_Parts:C0805C104K1RACTU
- added FADER: MF100T, Slider:SM10001NKA0X-HA1
- added IC5: TB6612FNG,C,8,EL, SamacSys_Parts:TB6612FNG,C,8,EL
- added LED1, LED2: 150080GS75000, SamacSys_Parts:150080GS75000
- C5, C6: value 100nF -> 10uF; device SamacSys_Parts:C0805C104K1RACTU -> SamacSys_Parts:T491A106M016AT7280
- C7: device SamacSys_Parts:EEE-HB1C100R -> SamacSys_Parts:T491A106M016AT7280
- C8: value 10uF -> 100nF; device SamacSys_Parts:EEE-HB1C100R -> SamacSys_Parts:C0805C104K1RACTU
- R3: value 100K -> 470R
- renumbered IO1 to SV1, IO2 to SV2, NEO to SV3, TOUCH to LED3, U$2 to LOGO, UPDI to SV4, X1 to SV5
Connections:
- removed net ENABLE: IC1.PB3, IC3.ENABLE_1, IC3.ENABLE_2
- removed net LB-LED: IC1.PA1, LB-LED.K
- removed net MOT-A: IC1.PA5, IC3.INPUT_1, IC3.INPUT_4
- removed net MOT-B: IC1.PA6, IC3.INPUT_2, IC3.INPUT_3
- removed net N$5: LB-LED.A, R7.1
- new net AIN1: IC1.PA5, IC5.AIN1
- new net AIN2: IC1.PA6, IC5.AIN2
- new net PWM: IC1.PB3, IC5.PWMA
- new net STBY: IC1.PA1, IC5.STBY
- net +5V: now also C5.+, C6.+, C8.1, FADER.3, IC5.VCC; no longer C6.2, C8.+, IC3.VSS, R3.1, R7.2, U$1.3
- net 9V-DRIVE: now also C9.1, IC5.VM1, IC5.VM2, IC5.VM3, SV1.6, SV2.6; no longer C5.2, IC3.VS, SV1.1, SV2.1
- net D-OUT: now also R3.1; no longer R9.1
- net GND: now also C5.-, C6.-, C8.2, C9.2, FADER.1, IC5.GND, IC5.PGND1_1, IC5.PGND1_2, IC5.PGND2_1, IC5.PGND2_2, LED1.K, LED2.K; no longer +5V.K, +9V.K, C5.1, C6.1, C8.-, IC3.GND_1, IC3.GND_2, IC3.GND_3, IC3.GND_4, IC3.GND_5, IC3.GND_6, IC3.GND_7, IC3.GND_8, U$1.1
- net INR: now also SV1.1, SV2.1; no longer R3.2, SV1.6, SV2.6
- net MOT+: now also FADER.A, IC5.AO1_1, IC5.AO1_2; no longer IC3.OUTPUT_1, IC3.OUTPUT_4, U$1.A
- net MOT-: now also FADER.B, IC5.AO2_1, IC5.AO2_2; no longer IC3.OUTPUT_2, IC3.OUTPUT_3, U$1.B
- net N$2: now also LED1.A; no longer +5V.A
- net N$3: now also LED2.A; no longer +9V.A
- net N$6: now also R3.2; no longer R9.2
- net SERVOTRACK: now also FADER.2; no longer U$1.2
- net TOUCH: now also FADER.T; no longer U$1.T
Other:
- moved on the sheet: C7, R2, R3, R6
