File: PCB/Eagel/ServoFaderTB6612.V.1.0.sch (EAGLE design)
At the start: 29 parts, among them IC1 ATTINY804-SSNR, IC2 AT42QT1010, IC4 SN74LVC1G14DBVR, IC5 TB6612FNG,C,8,EL

Commit message: update
Parts:
- C3: device SamacSys_Parts:C0805C104K1RACTU -> SamacSys_Parts:C0805C223K5RAC7210
- C4: device SamacSys_Parts:C0805C333K4RACTU -> SamacSys_Parts:C0805C223K5RAC7210
Other:
- moved on the sheet: C1, C2, C3, C4, C5, C6, C7, C8, C9, FADER, IC1, IC2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

Commit message: Update Pin PB3
Connections:
- removed net N$6: IC1.PB2, R3.2
- new net N$5: IC1.PA6, R3.2
- net AIN2: now also IC1.PB3; no longer IC1.PA6
- net PWM: now also IC1.PB2; no longer IC1.PB3
Other:
- moved on the sheet: R3
Changed lines of the file:
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@@
 </instance>
 <instance part="LOGO" gate="G$1" x="182.372" y="-110.236" smashed="yes"/>
-<instance part="R3" gate="G$1" x="7.62" y="2.54" smashed="yes" grouprefs="MICROCONTROLLER">
-<attribute name="NAME" x="3.81" y="-1.0414" size="1.778" layer="95"/>
-<attribute name="VALUE" x="8.89" y="-0.762" size="1.778" layer="96"/>
+<instance part="R3" gate="G$1" x="5.08" y="10.16" smashed="yes" grouprefs="MICROCONTROLLER">
+<attribute name="NAME" x="1.27" y="11.6586" size="1.778" layer="95"/>
+<attribute name="VALUE" x="6.35" y="11.938" size="1.778" layer="96"/>
 </instance>
 <instance part="SV3" gate="G$1" x="-139.7" y="-88.9" smashed="yes" rot="R90">
@@
 <net name="PWM" class="0">
 <segment>
-<pinref part="IC1" gate="G$1" pin="PB3"/>
-<wire x1="25.4" y1="5.08" x2="20.32" y2="5.08" width="0.1524" layer="91" grouprefs="MICROCONTROLLER"/>
-<label x="20.32" y="5.08" size="1.016" layer="95" rot="R180" xref="yes" grouprefs="MICROCONTROLLER"/>
+<label x="20.32" y="2.54" size="1.016" layer="95" rot="R180" xref="yes" grouprefs="MICROCONTROLLER"/>
+<pinref part="IC1" gate="G$1" pin="PB2"/>
+<wire x1="25.4" y1="2.54" x2="20.32" y2="2.54" width="0.1524" layer="91"/>
 </segment>
 <segment>
@@
 <net name="AIN2" class="0">
 <segment>
-<pinref part="IC1" gate="G$1" pin="PA6"/>
-<wire x1="25.4" y1="10.16" x2="20.32" y2="10.16" width="0.1524" layer="91" grouprefs="MICROCONTROLLER"/>
-<label x="20.32" y="10.16" size="1.016" layer="95" rot="R180" xref="yes" grouprefs="MICROCONTROLLER"/>
+<label x="20.32" y="5.08" size="1.016" layer="95" rot="R180" xref="yes" grouprefs="MICROCONTROLLER"/>
+<pinref part="IC1" gate="G$1" pin="PB3"/>
+<wire x1="20.32" y1="5.08" x2="25.4" y2="5.08" width="0.1524" layer="91"/>
 </segment>
 <segment>
@@
 </segment>
 </net>
-<net name="N$6" class="0">
-<segment>
-<pinref part="R3" gate="G$1" pin="2"/>
-<pinref part="IC1" gate="G$1" pin="PB2"/>
-<wire x1="12.7" y1="2.54" x2="25.4" y2="2.54" width="0.1524" layer="91" grouprefs="MICROCONTROLLER"/>
-</segment>
-</net>
 <net name="D-OUT" class="0">
 <segment>
 <pinref part="R3" gate="G$1" pin="1"/>
-<wire x1="2.54" y1="2.54" x2="0" y2="2.54" width="0.1524" layer="91" grouprefs="MICROCONTROLLER"/>
-<label x="0" y="2.54" size="1.016" layer="95" rot="R180" xref="yes" grouprefs="MICROCONTROLLER"/>
+<wire x1="0" y1="10.16" x2="-2.54" y2="10.16" width="0.1524" layer="91" grouprefs="MICROCONTROLLER"/>
+<label x="-2.54" y="10.16" size="1.016" layer="95" rot="R180" xref="yes" grouprefs="MICROCONTROLLER"/>
 </segment>
 <segment>
@@
 </segment>
 </net>
+<net name="N$5" class="0">
+<segment>
+<pinref part="IC1" gate="G$1" pin="PA6"/>
+<pinref part="R3" gate="G$1" pin="2"/>
+<wire x1="10.16" y1="10.16" x2="25.4" y2="10.16" width="0.1524" layer="91"/>
+</segment>
+</net>

Commit message: Update
Motorsteuerung mit ABS eingefügt
Parts:
- IC1: value ATTINY804-SSNR -> ATTINY1604-SSN; device SamacSys_Parts:ATTINY804-SSNR -> SamacSys_Parts:ATTINY1604-SSN
Changed lines of the file:
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@@
 <parts>
 <part name="FADER" library="Slider" deviceset="SM10001NKA0X-HA1" device="" value="MF100T"/>
-<part name="IC1" library="SamacSys_Parts" deviceset="ATTINY804-SSNR" device=""/>
+<part name="IC1" library="SamacSys_Parts" deviceset="ATTINY1604-SSN" device=""/>
 <part name="IC2" library="SamacSys_Parts" deviceset="AT42QT1010-TSHR" device="" value="AT42QT1010"/>
 <part name="LED1" library="SamacSys_Parts" deviceset="150080GS75000" device=""/>
